File: hardware/eagle_v7_6/p25rx_display_rev3.brd (EAGLE design)
At the start: 104.7 x 52 mm, 79 parts, among them J1 SJ-3523, J2 USB4085, J3 1050170001, J4 SJ-3523, J5 SF: PRT-10361, J7 SF: PRT-10361, Q1 IRFR5305, Q16 2N7002, SW2 CHS-01TA, U1 LCD24, U2 IS31AP4991A-GRLS2-TR, U4 STM32H743ZIT6, U5 CS4344, U6 MCP1826ST-3302E/DB, X2 8MHZ

Commit message: update notes on schematic regarding D2
Parts:
- D2: value (none) -> zero_ohm
Changed lines of the file:
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@@
 <attribute name="NAME" x="415.45976875" y="-8.39966875" size="0.6096" layer="25" rot="R90"/>
 </element>
-<element name="D2" library="diode" package="SMB" value="" x="399.4658" y="-28.067" smashed="yes">
+<element name="D2" library="diode" package="SMB" value="zero_ohm" x="399.4658" y="-28.067" smashed="yes">
 <attribute name="NAME" x="398.8054" y="-26.0096" size="0.6096" layer="25"/>
 <attribute name="VALUE" x="397.3068" y="-31.496" size="1.27" layer="27"/>
